File: System Memory Board.kicad_sch (KiCad schematic)
At the start: 23 parts, among them P300 AMP 5-102871-1, U55 74ALS245, U56 74ALS245, U57 SN74S734, U58 74F32

Commit message: separate Write Enable signals for bank 2 and bank 3/4
Connections:
- net ~{WE34}: now reaches P300.a4 (Pin_a4)
- net ~{WE34}: now also R5.1
- net ~{WE} renamed ~{WE2}
- net ~{WE2}: no longer R5.1
Other:
- moved on the sheet: C70, C71, C72, C73, C74, R4, R5, R6, R7, R8

Commit message: connect last few nets
Connections:
- net MA6: now also Z1.2 (R1)
- net VCC: now also Z1.1 (common)
- no-connect marks 0 -> 6
Changed lines of the file:
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@@
 		(color 0 0 0 0)
 	)
+	(no_connect
+		(at 106.68 27.94)
+	)
+	(no_connect
+		(at 243.84 33.02)
+	)
+	(no_connect
+		(at 63.5 27.94)
+	)
+	(no_connect
+		(at 132.08 27.94)
+	)
+	(no_connect
+		(at 243.84 30.48)
+	)
+	(no_connect
+		(at 231.14 30.48)
+	)
 	(wire
 		(pts
@@
 	(wire
 		(pts
+			(xy 43.18 27.94) (xy 43.18 35.56)
+		)
+		(stroke
+			(width 0)
+			(type default)
+		)
+	)
+	(wire
+		(pts
 			(xy 106.68 88.9) (xy 109.22 88.9)
 		)
@@
 					(unit 1)
 				)
+			)
+		)
+	)
+	(symbol
+		(lib_id "power:VCC")
+		(at 43.18 17.78 0)
+		(unit 1)
+		(exclude_from_sim no)
+		(in_bom yes)
+		(on_board yes)
+		(dnp no)
+		(fields_autoplaced yes)
+		(property "Reference" "#PWR070"
+			(at 43.18 21.59 0)
+			(effects
+				(font
+					(size 1.27 1.27)
+				)
+				(hide yes)
+			)
+		)
+		(property "Value" "VCC"
+			(at 43.18 13.97 0)
+			(effects
+				(font
+					(size 1.27 1.27)
+				)
+			)
+		)
+		(property "Footprint" ""
+			(at 43.18 17.78 0)
+			(effects
+				(font
+					(size 1.27 1.27)
+				)
+				(hide yes)
+			)
+		)
+		(property "Datasheet" ""
+			(at 43.18 17.78 0)
+			(effects
+				(font
+					(size 1.27 1.27)
+				)
+				(hide yes)
+			)
+		)
+		(property "Description" "Power symbol creates a global label with name \"VCC\""
+			(at 43.18 17.78 0)
+			(effects
+				(font
+					(size 1.27 1.27)
+				)
+				(hide yes)
+			)
+		)
+		(pin "1"
+		)
+		(instances
+			(project "System Memory Board"
+				(path "/5d4fb4c3-1130-42ed-b8b4-cc3440786f60"
+					(reference "#PWR070")
+					(unit 1)
+				)

Commit message: updates to match compaq design
Parts:
- U55, U56, U57: footprint Package_DIP:DIP-20_W7.62mm -> Library:DIP-20_W7.62mm
- U58: footprint Package_DIP:DIP-14_W7.62mm -> Library:DIP-14_W7.62mm
Changed lines of the file:
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@@
 			)
 		)
-		(property "Footprint" "Package_DIP:DIP-14_W7.62mm"
+		(property "Footprint" "Library:DIP-14_W7.62mm"
 			(at 198.12 88.9 0)
 			(effects
@@
 			)
 		)
-		(property "Footprint" "Package_DIP:DIP-20_W7.62mm"
+		(property "Footprint" "Library:DIP-20_W7.62mm"
 			(at 177.8 121.92 0)
 			(effects
@@
 			)
 		)
-		(property "Footprint" "Package_DIP:DIP-20_W7.62mm"
+		(property "Footprint" "Library:DIP-20_W7.62mm"
 			(at 233.68 121.92 0)
 			(effects
@@
 			)
 		)
-		(property "Footprint" "Package_DIP:DIP-14_W7.62mm"
+		(property "Footprint" "Library:DIP-14_W7.62mm"
 			(at 233.68 152.4 0)
 			(effects
@@
 			)
 		)
-		(property "Footprint" "Package_DIP:DIP-14_W7.62mm"
+		(property "Footprint" "Library:DIP-14_W7.62mm"
 			(at 198.12 78.74 0)
 			(effects
@@
 			)
 		)
-		(property "Footprint" "Package_DIP:DIP-20_W7.62mm"
+		(property "Footprint" "Library:DIP-20_W7.62mm"
 			(at 177.8 45.72 0)
 			(effects
