File: bank2.kicad_sch (KiCad schematic)
At the start: 18 parts, among them U15 41256, U16 41256, U23 41256, U24 41256, U31 41256, U32 41256, U39 41256, U40 41256, U47 41256, U48 41256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

Commit message: updates to match compaq design
Parts:
- U15, U16, U23, U24, U31, U32, U39, U40, U47, U48, U49, U50, U51, U52, U53, U54, U7, U8: footprint Package_DIP:DIP-16_W7.62mm -> Library:DIP-16_W7.62mm
Changed lines of the file:
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@@
 			)
 		)
-		(property "Footprint" "Package_DIP:DIP-16_W7.62mm"
+		(property "Footprint" "Library:DIP-16_W7.62mm"
 			(at 208.28 125.73 0)
 			(effects
@@
 			)
 		)
-		(property "Footprint" "Package_DIP:DIP-16_W7.62mm"
+		(property "Footprint" "Library:DIP-16_W7.62mm"
 			(at 147.32 46.99 0)
 			(effects
@@
 			)
 		)
-		(property "Footprint" "Package_DIP:DIP-16_W7.62mm"
+		(property "Footprint" "Library:DIP-16_W7.62mm"
 			(at 167.64 46.99 0)
 			(effects
@@
 			)
 		)
-		(property "Footprint" "Package_DIP:DIP-16_W7.62mm"
+		(property "Footprint" "Library:DIP-16_W7.62mm"
 			(at 236.22 125.73 0)
 			(effects
@@
 			)
 		)
-		(property "Footprint" "Package_DIP:DIP-16_W7.62mm"
+		(property "Footprint" "Library:DIP-16_W7.62mm"
 			(at 187.96 46.99 0)
 			(effects
@@
 			)
 		)
-		(property "Footprint" "Package_DIP:DIP-16_W7.62mm"
+		(property "Footprint" "Library:DIP-16_W7.62mm"
 			(at 167.64 125.73 0)
 			(effects
@@
 			)
 		)
-		(property "Footprint" "Package_DIP:DIP-16_W7.62mm"
+		(property "Footprint" "Library:DIP-16_W7.62mm"
 			(at 187.96 125.73 0)
 			(effects
@@
 			)
 		)
-		(property "Footprint" "Package_DIP:DIP-16_W7.62mm"
+		(property "Footprint" "Library:DIP-16_W7.62mm"
 			(at 106.68 46.99 0)
 			(effects
@@
 			)
 		)
-		(property "Footprint" "Package_DIP:DIP-16_W7.62mm"
+		(property "Footprint" "Library:DIP-16_W7.62mm"
 			(at 66.04 125.73 0)
 			(effects
@@
 			)
 		)
-		(property "Footprint" "Package_DIP:DIP-16_W7.62mm"
+		(property "Footprint" "Library:DIP-16_W7.62mm"
 			(at 86.36 125.73 0)
 			(effects
@@
 			)
 		)
-		(property "Footprint" "Package_DIP:DIP-16_W7.62mm"
+		(property "Footprint" "Library:DIP-16_W7.62mm"
 			(at 127 125.73 0)
 			(effects
@@
 			)
 		)
-		(property "Footprint" "Package_DIP:DIP-16_W7.62mm"
+		(property "Footprint" "Library:DIP-16_W7.62mm"
 			(at 106.68 125.73 0)
 			(effects
@@
 			)
 		)
-		(property "Footprint" "Package_DIP:DIP-16_W7.62mm"
+		(property "Footprint" "Library:DIP-16_W7.62mm"
 			(at 86.36 46.99 0)
 			(effects
@@
 			)
 		)
-		(property "Footprint" "Package_DIP:DIP-16_W7.62mm"
+		(property "Footprint" "Library:DIP-16_W7.62mm"
 			(at 236.22 46.99 0)
 			(effects
@@
 			)
 		)
-		(property "Footprint" "Package_DIP:DIP-16_W7.62mm"
+		(property "Footprint" "Library:DIP-16_W7.62mm"
 			(at 208.28 46.99 0)
 			(effects
@@
 			)
 		)
-		(property "Footprint" "Package_DIP:DIP-16_W7.62mm"
+		(property "Footprint" "Library:DIP-16_W7.62mm"
 			(at 147.32 125.73 0)
 			(effects
@@
 			)
 		)
-		(property "Footprint" "Package_DIP:DIP-16_W7.62mm"
+		(property "Footprint" "Library:DIP-16_W7.62mm"
 			(at 127 46.99 0)
 			(effects
@@
 			)
 		)
-		(property "Footprint" "Package_DIP:DIP-16_W7.62mm"
+		(property "Footprint" "Library:DIP-16_W7.62mm"
 			(at 66.04 46.99 0)
 			(effects
