File: bank4.kicad_sch (KiCad schematic)
At the start: 18 parts, among them U1 41256, U10 41256, U11 41256, U17 41256, U18 41256, U19 41256, U2 41256, U25 41256, U26 41256, U27 41256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

Commit message: updates to match compaq design
Parts:
- U1, U10, U11, U17, U18, U19, U2, U25, U26, U27, U3, U33, U34, U35, U41, U42, U43, U9: footprint Package_DIP:DIP-16_W7.62mm -> Library:DIP-16_W7.62mm_Socket
Changed lines of the file:
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@@
 			)
 		)
-		(property "Footprint" "Package_DIP:DIP-16_W7.62mm"
+		(property "Footprint" "Library:DIP-16_W7.62mm_Socket"
 			(at 208.28 125.73 0)
 			(effects
@@
 			)
 		)
-		(property "Footprint" "Package_DIP:DIP-16_W7.62mm"
+		(property "Footprint" "Library:DIP-16_W7.62mm_Socket"
 			(at 147.32 46.99 0)
 			(effects
@@
 			)
 		)
-		(property "Footprint" "Package_DIP:DIP-16_W7.62mm"
+		(property "Footprint" "Library:DIP-16_W7.62mm_Socket"
 			(at 167.64 46.99 0)
 			(effects
@@
 			)
 		)
-		(property "Footprint" "Package_DIP:DIP-16_W7.62mm"
+		(property "Footprint" "Library:DIP-16_W7.62mm_Socket"
 			(at 236.22 125.73 0)
 			(effects
@@
 			)
 		)
-		(property "Footprint" "Package_DIP:DIP-16_W7.62mm"
+		(property "Footprint" "Library:DIP-16_W7.62mm_Socket"
 			(at 187.96 46.99 0)
 			(effects
@@
 			)
 		)
-		(property "Footprint" "Package_DIP:DIP-16_W7.62mm"
+		(property "Footprint" "Library:DIP-16_W7.62mm_Socket"
 			(at 167.64 125.73 0)
 			(effects
@@
 			)
 		)
-		(property "Footprint" "Package_DIP:DIP-16_W7.62mm"
+		(property "Footprint" "Library:DIP-16_W7.62mm_Socket"
 			(at 187.96 125.73 0)
 			(effects
@@
 			)
 		)
-		(property "Footprint" "Package_DIP:DIP-16_W7.62mm"
+		(property "Footprint" "Library:DIP-16_W7.62mm_Socket"
 			(at 106.68 46.99 0)
 			(effects
@@
 			)
 		)
-		(property "Footprint" "Package_DIP:DIP-16_W7.62mm"
+		(property "Footprint" "Library:DIP-16_W7.62mm_Socket"
 			(at 66.04 125.73 0)
 			(effects
@@
 			)
 		)
-		(property "Footprint" "Package_DIP:DIP-16_W7.62mm"
+		(property "Footprint" "Library:DIP-16_W7.62mm_Socket"
 			(at 86.36 125.73 0)
 			(effects
@@
 			)
 		)
-		(property "Footprint" "Package_DIP:DIP-16_W7.62mm"
+		(property "Footprint" "Library:DIP-16_W7.62mm_Socket"
 			(at 127 125.73 0)
 			(effects
@@
 			)
 		)
-		(property "Footprint" "Package_DIP:DIP-16_W7.62mm"
+		(property "Footprint" "Library:DIP-16_W7.62mm_Socket"
 			(at 106.68 125.73 0)
 			(effects
@@
 			)
 		)
-		(property "Footprint" "Package_DIP:DIP-16_W7.62mm"
+		(property "Footprint" "Library:DIP-16_W7.62mm_Socket"
 			(at 86.36 46.99 0)
 			(effects
@@
 			)
 		)
-		(property "Footprint" "Package_DIP:DIP-16_W7.62mm"
+		(property "Footprint" "Library:DIP-16_W7.62mm_Socket"
 			(at 236.22 46.99 0)
 			(effects
@@
 			)
 		)
-		(property "Footprint" "Package_DIP:DIP-16_W7.62mm"
+		(property "Footprint" "Library:DIP-16_W7.62mm_Socket"
 			(at 208.28 46.99 0)
 			(effects
@@
 			)
 		)
-		(property "Footprint" "Package_DIP:DIP-16_W7.62mm"
+		(property "Footprint" "Library:DIP-16_W7.62mm_Socket"
 			(at 147.32 125.73 0)
 			(effects
@@
 			)
 		)
-		(property "Footprint" "Package_DIP:DIP-16_W7.62mm"
+		(property "Footprint" "Library:DIP-16_W7.62mm_Socket"
 			(at 127 46.99 0)
 			(effects
@@
 			)
 		)
-		(property "Footprint" "Package_DIP:DIP-16_W7.62mm"
+		(property "Footprint" "Library:DIP-16_W7.62mm_Socket"
 			(at 66.04 46.99 0)
 			(effects
