File: misc.kicad_sch (KiCad schematic)
At the start: 70 parts, among them U58 74F32

Commit message: connect last few nets
Connections:
- no-connect marks 0 -> 3
Changed lines of the file:
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@@
 		(color 0 0 0 0)
+	)
+	(no_connect
+		(at 213.36 40.64)
+	)
+	(no_connect
+		(at 228.6 38.1)
+	)
+	(no_connect
+		(at 213.36 35.56)
 	)
 	(wire

Commit message: updates to match compaq design
Parts:
- C27, C29, C32, C33, C34, C35, C36, C37, C38, C39: footprint Capacitor_THT:CP_Radial_Tantal_D4.5mm_P5.00mm -> Library:CP_Radial_Tantal_D4.5mm_P5.00mm
- U58: footprint Package_DIP:DIP-14_W7.62mm -> Library:DIP-14_W7.62mm
Changed lines of the file:
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@@
 			)
 		)
-		(property "Footprint" "Capacitor_THT:CP_Radial_Tantal_D4.5mm_P5.00mm"
+		(property "Footprint" "Library:CP_Radial_Tantal_D4.5mm_P5.00mm"
 			(at 155.9052 83.82 0)
 			(effects
@@
 			)
 		)
-		(property "Footprint" "Capacitor_THT:CP_Radial_Tantal_D4.5mm_P5.00mm"
+		(property "Footprint" "Library:CP_Radial_Tantal_D4.5mm_P5.00mm"
 			(at 125.4252 83.82 0)
 			(effects
@@
 			)
 		)
-		(property "Footprint" "Package_DIP:DIP-14_W7.62mm"
+		(property "Footprint" "Library:DIP-14_W7.62mm"
 			(at 220.98 38.1 0)
 			(effects
@@
 			)
 		)
-		(property "Footprint" "Package_DIP:DIP-14_W7.62mm"
+		(property "Footprint" "Library:DIP-14_W7.62mm"
 			(at 205.74 137.16 0)
 			(effects
@@
 			)
 		)
-		(property "Footprint" "Capacitor_THT:CP_Radial_Tantal_D4.5mm_P5.00mm"
+		(property "Footprint" "Library:CP_Radial_Tantal_D4.5mm_P5.00mm"
 			(at 84.7852 83.82 0)
 			(effects
@@
 			)
 		)
-		(property "Footprint" "Capacitor_THT:CP_Radial_Tantal_D4.5mm_P5.00mm"
+		(property "Footprint" "Library:CP_Radial_Tantal_D4.5mm_P5.00mm"
 			(at 135.5852 83.82 0)
 			(effects
@@
 			)
 		)
-		(property "Footprint" "Capacitor_THT:CP_Radial_Tantal_D4.5mm_P5.00mm"
+		(property "Footprint" "Library:CP_Radial_Tantal_D4.5mm_P5.00mm"
 			(at 176.2252 68.58 0)
 			(effects
@@
 			)
 		)
-		(property "Footprint" "Capacitor_THT:CP_Radial_Tantal_D4.5mm_P5.00mm"
+		(property "Footprint" "Library:CP_Radial_Tantal_D4.5mm_P5.00mm"
 			(at 105.1052 83.82 0)
 			(effects
@@
 			)
 		)
-		(property "Footprint" "Capacitor_THT:CP_Radial_Tantal_D4.5mm_P5.00mm"
+		(property "Footprint" "Library:CP_Radial_Tantal_D4.5mm_P5.00mm"
 			(at 115.2652 83.82 0)
 			(effects
@@
 			)
 		)
-		(property "Footprint" "Capacitor_THT:CP_Radial_Tantal_D4.5mm_P5.00mm"
+		(property "Footprint" "Library:CP_Radial_Tantal_D4.5mm_P5.00mm"
 			(at 145.7452 83.82 0)
 			(effects
@@
 			)
 		)
-		(property "Footprint" "Capacitor_THT:CP_Radial_Tantal_D4.5mm_P5.00mm"
+		(property "Footprint" "Library:CP_Radial_Tantal_D4.5mm_P5.00mm"
 			(at 94.9452 83.82 0)
 			(effects
@@
 			)
 		)
-		(property "Footprint" "Capacitor_THT:CP_Radial_Tantal_D4.5mm_P5.00mm"
+		(property "Footprint" "Library:CP_Radial_Tantal_D4.5mm_P5.00mm"
 			(at 155.9052 68.58 0)
 			(effects
